File: Eagle Schematics/RobotArm.brd (EAGLE design)
At the start: 100 x 80 mm, 87 parts, among them J1 5A/28V, SW1 5A/28V

Commit message: I routed everything except for VCC. I am not sure how to proceed from here.
Parts:
- removed SERVO1, SERVO2, SERVO3, SERVO4, SERVO6: HK15298B, PiB_motors:1X03-VERT-MALE
- added SERVOINDEX, SERVOMIDDLE, SERVOPINKY, SERVORING, SERVOTHUMB: HK15298B, PiB_motors:1X03-VERT-MALE
- moved C34 249.2 mm to (37.3, 11.2), turned to 270 degrees
- moved C36 249.0 mm to (11.7, 11.2), turned to 270 degrees
- moved C35 247.2 mm to (21.6, 10.9), turned to 90 degrees
- moved C33 244.7 mm to (39.1, 11.2), turned to 270 degrees
- moved C29 223.7 mm to (29.0, 43.9), turned to 270 degrees
- moved C31 223.0 mm to (32.6, 30.0)
- moved C28 208.5 mm to (51.9, 36.6)
- moved C27 188.2 mm to (32.7, 32.8), turned to 180 degrees
- moved C19 153.9 mm to (29.4, 11.2), turned to 180 degrees
- moved C16 152.6 mm to (51.0, 29.2), turned to 180 degrees
- moved C32 151.4 mm to (48.0, 10.2), turned to 180 degrees
- moved C30 148.3 mm to (26.4, 43.9), turned to 270 degrees
- moved C18 139.1 mm to (15.1, 11.2)
- moved C12 127.4 mm to (11.5, 25.1), turned to 180 degrees
- moved C9 125.8 mm to (17.7, 35.6), turned to 180 degrees
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Connections:
- net 5V: now also SERVOINDEX.VCC, SERVOMIDDLE.VCC, SERVOPINKY.VCC, SERVORING.VCC, SERVOTHUMB.VCC; no longer SERVO1.VCC, SERVO2.VCC, SERVO3.VCC, SERVO4.VCC, SERVO6.VCC
- net N$1: now also SERVOTHUMB.SIG; no longer SERVO6.SIG
- net N$3: now also SERVOINDEX.SIG; no longer SERVO1.SIG
- net N$4: now also SERVOMIDDLE.SIG; no longer SERVO2.SIG
- net N$5: now also SERVORING.SIG; no longer SERVO3.SIG
- net N$6: now also SERVOPINKY.SIG; no longer SERVO4.SIG
- net NGND: now also SERVOINDEX.GND, SERVOMIDDLE.GND, SERVOPINKY.GND, SERVORING.GND, SERVOTHUMB.GND; no longer SERVO1.GND, SERVO2.GND, SERVO3.GND, SERVO4.GND, SERVO6.GND
Routing:
- net SERVO-MIDDLE: track 0.00 -> 67.4 mm
- net SERVO-INDEX: track 0.00 -> 62.9 mm
- net SERVO-PINKY: track 0.00 -> 48.8 mm
- net SERVO-THUMB: track 0.00 -> 46.7 mm
- net GND: track 0.00 -> 46.0 mm, vias 0 -> 29
- net SERVO-RING: track 0.00 -> 44.4 mm
- net RESET: track 0.00 -> 43.1 mm
- net PRESS-THUMB: track 0.00 -> 41.7 mm
- net N$10: track 0.00 -> 33.7 mm
- net PRESS-INDEX: track 0.00 -> 33.3 mm
- net MOSI: track 0.00 -> 32.6 mm
- net MISO: track 0.00 -> 31.6 mm
- net SCK: track 0.00 -> 28.0 mm
- net N$12: track 0.00 -> 27.6 mm
- net PRESS-PINKY: track 0.00 -> 25.9 mm
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- added copper zone on layer 16, net AGND
- added copper zone on layer 16, net GND
- added copper zone on layer 16, net NGND
Other:
- board size 100 x 80 mm -> 54.5 x 52.8 mm

Commit message: last update
Parts:
- moved C30 2.03 mm to (24.4, 43.9)
- moved C29 0.76 mm to (28.2, 43.9)
Routing:
- net VBAT: track 0.00 -> 73.9 mm, vias 0 -> 1
- net VCC: track 0.00 -> 55.9 mm
- net 5V: track 0.00 -> 33.8 mm
- net SERVO-RING: track 44.4 -> 50.8 mm
- net AVCC: track 0.00 -> 2.83 mm
- net NGND: track 14.8 -> 13.3 mm
- net GND: track 46.0 -> 47.4 mm, vias 29 -> 31
- net SERVO-PINKY: track 48.8 -> 50.1 mm
- net PB7: track 3.88 -> 3.19 mm
Other:
- outline, holes or cut-outs redrawn

Commit message: Massaged around some stuff.
Parts:
- removed D2: (no value), PiB_discrete_semiconductors:SODFL3516X170
- C13, C14, C15, C17, C2, C20, C21, C25, C3, C30, C4, C5, C6, C7: device PiB_capacitors:CAPC2012X95_SMD-0805@1 -> PiB_capacitors:CAPC2012X95_SMD-0805
- C23, C24: value 470uF/50V -> 1000uF/16V; device PiB_capacitors:_AE_PTH_DIA10-LS5-H22 -> PiB_capacitors:_AE_PTH_DIA8-LS3.5-H21.50
- C32, C33, C34, C35, C36: value 0.1uF/50V -> 10uF/25V; device PiB_capacitors:CAPC1005X55_SMD-0402 -> PiB_capacitors:CAPC2012X95_SMD-0805
- D1, D3: value (none) -> 1A/50V
- FSR1, FSR2, FSR3, FSR4, FSR5: value FSR -> 10K; device PiB:CONNECTOR_FSR -> PiB_sensors:_MOLEX-0530470210_VERT_PITCH-1.25MM
- MCU1: device PiB_ic_microcontrollers:VFQFN-64 -> PiB_ic_microcontrollers:QFN50P900X900X90-64
- R20, R21: value 1K -> 10K
- SERVOINDEX, SERVOMIDDLE, SERVOPINKY, SERVORING, SERVOTHUMB: value HK15298B -> MG90S; device PiB_motors:1X03-VERT-MALE -> PiB:1X03-VERT-MALE
- moved C18 22.4 mm to (34.2, 22.9), turned to 180 degrees
- moved FTDI1 16.4 mm to (3.81, 44.7)
- moved LIPO1 15.8 mm to (16.6, 11.8), turned to 0 degrees
- moved C24 13.5 mm to (4.57, 33.3)
- moved C8 12.7 mm to (10.8, 21.3)
- moved C23 12.2 mm to (4.57, 24.7)
- moved D3 11.4 mm to (35.0, 17.3)
- moved C20 10.3 mm to (34.3, 20.7), turned to 180 degrees
- moved NET_BRIDGE1 10.3 mm to (10.3, 5.21), flipped to the bottom, turned to 0 degrees
- moved FSR5 9.22 mm to (34.1, 50.3)
- moved FSR4 7.45 mm to (38.6, 50.3)
- moved C15 7.19 mm to (10.9, 23.6), turned to 180 degrees
- moved C21 6.28 mm to (39.5, 8.69)
- moved C12 6.11 mm to (16.8, 28.3), turned to 270 degrees
- moved FSR3 5.42 mm to (43.2, 50.3)
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Connections:
- removed net 3.3V: AVR_ISP1.VCC
- removed net N$21: MCU1.46
- removed net N$22: MCU1.47
- net AGND: now also MCU1.EP, MCU1.P$1, MCU1.P$2, MCU1.P$3, MCU1.P$4, MCU1.P$5, R1.2, R2.2, R3.2, R4.2, R5.2
- net GND: no longer R1.2, R2.2, R3.2, R4.2, R5.2
- net PRESS-INDEX: now also FSR2.2; no longer FSR2.-
- net PRESS-MIDDLE: now also FSR3.2; no longer FSR3.-
- net PRESS-PINKY: now also FSR5.2; no longer FSR5.-
- net PRESS-RING: now also FSR4.2; no longer FSR4.-
- net PRESS-THUMB: now also FSR1.2; no longer FSR1.-
- net RX0: now also MCU1.46
- net TX0: now also MCU1.47
- net VBAT: no longer D2.K
- net VCC: now also FSR1.1, FSR2.1, FSR3.1, FSR4.1, FSR5.1; no longer D2.A, FSR1.+, FSR2.+, FSR3.+, FSR4.+, FSR5.+, FTDI1.VCC
Routing:
- net GND: track 47.4 -> 67.3 mm, vias 31 -> 27
- net VBAT: track 73.9 -> 89.7 mm
- net AGND: track 9.40 -> 22.2 mm, vias 3 -> 7
- net PRESS-PINKY: track 25.9 -> 35.2 mm
- net 5V: track 33.8 -> 25.9 mm
- net VCC: track 55.9 -> 63.7 mm
- net SCK: track 28.0 -> 33.9 mm
- net MOSI: track 32.6 -> 38.4 mm
- net MISO: track 31.6 -> 35.4 mm
- net RESET: track 43.1 -> 46.2 mm
- net NGND: track 13.3 -> 10.6 mm, vias 11 -> 16
- net N$10: track 33.7 -> 32.1 mm
- net PRESS-THUMB: track 41.6 -> 43.0 mm
- net SERVO-RING: track 50.8 -> 51.9 mm
- net SERVO-PINKY: track 50.1 -> 51.1 mm
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- added copper zone on layer 1, net NGND
Other:
- board size 54.5 x 52.8 mm -> 54.5 x 52.6 mm

Commit message: reorganized
Parts:
- moved R17 25.8 mm to (18.5, 30.1), turned to 0 degrees
- moved R5 24.8 mm to (49.7, 48.6), turned to 90 degrees
- moved R16 23.7 mm to (18.5, 32.3), turned to 0 degrees
- moved LED1 23.5 mm to (14.6, 32.3), turned to 180 degrees
- moved C30 22.3 mm to (45.9, 38.1), turned to 0 degrees
- moved FSR1 20.2 mm to (52.3, 30.2), turned to 270 degrees
- moved LED2 19.0 mm to (14.6, 30.1), turned to 180 degrees
- moved C7 18.7 mm to (41.9, 26.3), turned to 90 degrees
- moved XTAL1 18.7 mm to (48.0, 25.5), turned to 270 degrees
- moved C6 18.6 mm to (44.5, 26.4), turned to 270 degrees
- moved C3 18.6 mm to (39.6, 26.3), turned to 270 degrees
- moved R4 18.5 mm to (49.6, 44.0), turned to 90 degrees
- moved FSR5 18.3 mm to (52.2, 48.4), turned to 270 degrees
- moved C27 18.1 mm to (14.6, 34.5)
- moved R1 16.9 mm to (49.6, 30.7), turned to 90 degrees
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Routing:
- net VCC: track 63.7 -> 127.2 mm, vias 0 -> 12
- net 5V: track 25.9 -> 80.4 mm
- net TX0: track 0.00 -> 50.6 mm, vias 0 -> 2
- net RX0: track 0.00 -> 47.0 mm, vias 0 -> 2
- net VBAT: track 89.7 -> 60.7 mm, vias 1 -> 2
- net PRESS-THUMB: track 43.0 -> 16.6 mm
- net N$12: track 27.8 -> 3.10 mm
- net N$11: track 25.9 -> 3.08 mm
- net SERVO-PINKY: track 51.1 -> 28.9 mm
- net +: track 0.00 -> 22.0 mm
- net SERVO-RING: track 51.9 -> 30.2 mm
- net MISO: track 35.4 -> 13.8 mm
- net AVCC: track 2.83 -> 23.9 mm, vias 0 -> 2
- net MOSI: track 38.4 -> 18.3 mm
- net PB6: track 3.42 -> 22.9 mm, vias 0 -> 2
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Other:
- board size 54.5 x 52.6 mm -> 54.6 x 50.8 mm

Commit message: Hopefully not too much to change
Parts:
- moved L2 21.1 mm to (41.8, 35.8)
- moved C3 3.87 mm to (43.3, 27.4), turned to 0 degrees
- moved C25 2.77 mm to (14.3, 39.5)
- moved C29 2.34 mm to (41.8, 38.2)
- moved C27 2.33 mm to (14.3, 36.8)
- moved C14 2.30 mm to (23.2, 24.7)
- moved C1 2.11 mm to (18.5, 43.3)
- moved C6 2.03 mm to (44.6, 24.3)
- moved C7 2.01 mm to (42.0, 24.3)
- moved LED1 1.65 mm to (14.4, 33.9)
- moved C12 1.39 mm to (23.2, 21.6)
- moved LED2 1.13 mm to (14.5, 31.2)
- moved C24 1.09 mm to (7.91, 34.2)
- moved C15 1.02 mm to (10.5, 28.9)
- moved LED3 1.02 mm to (14.5, 28.9)
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Routing:
- net AVCC: track 23.9 -> 11.0 mm, vias 2 -> 3
- net VCC: track 127.2 -> 135.8 mm, vias 12 -> 13
- net AGND: track 24.8 -> 32.4 mm, vias 10 -> 12
- net RESET: track 47.0 -> 39.7 mm, vias 6 -> 8
- net PRESS-MIDDLE: track 20.3 -> 25.0 mm
- net GND: track 67.6 -> 63.8 mm, vias 38 -> 36
- net PRESS-RING: track 21.9 -> 24.4 mm
- net TX0: track 50.6 -> 52.8 mm
- net PRESS-PINKY: track 26.7 -> 28.8 mm
- net N$9: track 15.3 -> 17.4 mm
- net N$14: track 5.40 -> 6.99 mm
- net RX0: track 47.0 -> 48.3 mm, vias 2 -> 4
- net VBAT: track 60.7 -> 61.9 mm
- net N$2: track 1.88 -> 2.80 mm
- net SCK: track 15.8 -> 16.8 mm
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
Commit message: jesus help me
Routing:
- net VBAT: track 61.9 -> 59.9 mm
- net PRESS-PINKY: track 28.8 -> 27.3 mm
- net VCC: track 135.8 -> 136.9 mm, vias 13 -> 12

Commit message: Create antenna CKTry.
Parts:
- moved D1 17.2 mm to (9.02, 42.1), turned to 180 degrees
- moved R20 13.3 mm to (9.47, 39.7), turned to 180 degrees
- moved FSR5 7.50 mm to (46.3, 43.8)
- moved R5 7.50 mm to (43.7, 44.0)
- moved C10 6.60 mm to (28.4, 35.8), turned to 0 degrees
- moved ANT1 4.13 mm to (31.7, 41.9)
- moved C11 1.19 mm to (28.4, 37.7), turned to 0 degrees
Connections:
- net AGND: now also BALUN1.5, C10.1, C11.1, MCU1.10, MCU1.7
- net GND: no longer BALUN1.5, C10.1, C11.1, MCU1.10, MCU1.7
Routing:
- net AGND: track 32.4 -> 20.2 mm, vias 12 -> 25
- net RESET: track 39.7 -> 51.4 mm, vias 8 -> 6
- net PRESS-PINKY: track 27.3 -> 18.8 mm
- net N$17: track 8.82 -> 1.89 mm
- net GND: track 63.8 -> 57.9 mm, vias 36 -> 32
- net N$16: track 5.49 -> 1.81 mm
- net PRESS-MIDDLE: track 24.6 -> 22.1 mm
- net VCC: track 136.9 -> 138.9 mm, vias 12 -> 10
- net SERVO-PINKY: track 29.1 -> 31.0 mm
- net SERVO-RING: track 30.9 -> 32.3 mm
- net SERVO-MIDDLE: track 61.3 -> 62.2 mm
- net SERVO-INDEX: track 52.4 -> 53.3 mm
- net SERVO-THUMB: track 42.4 -> 43.2 mm
- added copper zone on layer 1, net AGND
- added copper zone on layer 1, net N$17
Other:
- board size 54.6 x 50.8 mm -> 54.5 x 46 mm

Commit message: thank you so much Colin!
Parts:
- moved C1 9.91 mm to (8.54, 43.1)
- moved R20 9.18 mm to (18.4, 42.0)
- moved D1 4.57 mm to (13.6, 42.2), turned to 0 degrees
- moved R4 1.02 mm to (49.6, 43.0)
- moved R3 0.76 mm to (49.6, 38.6)
- moved R2 0.25 mm to (49.6, 34.6)
Routing:
- net N$10: track 15.5 -> 5.70 mm
- net VCC: track 138.9 -> 145.7 mm, vias 10 -> 12
- net AVCC: track 10.7 -> 9.31 mm, vias 3 -> 2
- net RESET: track 51.4 -> 50.1 mm
- net AGND: track 20.2 -> 21.0 mm
- net PRESS-MIDDLE: track 22.1 -> 22.8 mm
- net PRESS-RING: track 24.4 -> 23.8 mm
