File: Eagle Schematics/RobotArm.brd (EAGLE design)
At the start: 54.5 x 46 mm, 86 parts, among them J1 5A/28V, SW1 5A/28V

Commit message: Please check changes and order this piece
Routing:
- net VCC: track 145.7 -> 144.5 mm, vias 12 -> 13
- net VBAT: track 59.7 -> 60.2 mm
