File: Eagle /TouchGlove.sch (EAGLE design)
At the start: 77 parts, among them Q1 SI2302CDS 2.9A/20V, Q2 SI2302CDS 2.9A/20V, Q3 SI2302CDS 2.9A/20V, Q4 SI2302CDS 2.9A/20V, Q5 SI2302CDS 2.9A/20V, SW1 300mA/4V, Y1 16 MHz

Commit message: Rotated that shitty chip.
Parts:
- removed D6: 1A/50V, PiB_discrete_semiconductors:DIODE_GENERAL-PURPOSE_SMD_GP_1A-50V
- removed MOTOR1, MOTOR2, MOTOR3, MOTOR4, MOTOR5: (no value), PiB:MOTOR_PADSPTH
- added VIBE1, VIBE2, VIBE3, VIBE4, VIBE5: Molex VERT 1.25mm pitch, PiB_actuators:VIBE-MOTOR_CONNECTOR_0530470210_VERT-MALE_PITCH-1.25MM
- FLEX1, FLEX2, FLEX3, FLEX4, FLEX5: device PiB:FLEX-SENSOR10K_2.2IN -> PiB_sensors:FLEX_SENSOR_0530470210_VERT-MALE_PITCH-1.25MM
- VREG-MCU: device PiB_ic_power:VREG_TPS76833_ULDO_FAST-TRANSIENT_1A-3.3VTPS76833QDR_1A-3.3V -> PiB_ic_power:VREG_TPS768XX_ULDO_FAST-TRANSIENT_TPS76833QDR_1A-3.3V
Connections:
- net GND: now also C12.2, C13.2, C14.2, C15.2, C16.2, C17.2, C18.2, R17.1
- net N$1: now also VIBE1.-; no longer MOTOR1.V-
- net N$2: now also VIBE2.-; no longer MOTOR2.V-
- net N$24: no longer D6.K
- net N$3: now also VIBE3.-; no longer MOTOR3.V-
- net N$4: now also VIBE4.-; no longer MOTOR4.V-
- net N$5: now also VIBE5.-; no longer MOTOR5.V-
- net NGND: no longer C12.2, C13.2, C14.2, C15.2, C16.2, C17.2, C18.2, R17.1
- net VCC: now also VIBE1.+, VIBE2.+, VIBE3.+, VIBE4.+, VIBE5.+; no longer D6.A, MOTOR1.V+, MOTOR2.V+, MOTOR3.V+, MOTOR4.V+, MOTOR5.V+
Other:
- moved on the sheet: D1, D2, Q1, Q2, R11, R12, R6, R7

Commit message: Rev 1: Ready for fab.
Parts:
- removed C14: 100uF/10V, PiB_capacitors:100UF_CER_SMD-1210_16V-20%
- C1, C2: device PiB_capacitors:12PF_SMD-805_250V-5% -> PiB_capacitors:12PF_SMD-0805_250V-5%
- C3: value 22PF/250V -> 22pF/250V; device PiB_capacitors:22PF_SMD-805_250V-5% -> PiB_capacitors:22PF_CER_SMD-0805_250V-5%
- C4: value 0.75PF/100V -> 0.75pF/100V; device PiB_capacitors:0.75PF_SMD-805_100V-33% -> PiB_capacitors:0.75PF_CER_SMD-0805_100V-33%
- L1, L2: device PiB_inductors:10UH_SMD-805_0.5A-0.65OHM-10% -> PiB_inductors:10UH_SMD-0805_0.5A-0.65OHM-10%
- LED1: device PiB_leds:LED_SMD-0805_DISCRETE_GREEN -> PiB_leds:LED_SMD-0805_DISCRETE_GREEN_
- R1, R2, R3, R4, R5: device PiB_resistors:4.7KΩ_SMD-0805_1/8W-5% -> PiB_resistors:4.7KΩ_SMD-0805_1/8W_5%
- VREG-VIBE: device PiB_ic_power:VREG_LINEAR_FIXED_TL1963A-33_LDO_1.5A-3.3V -> PiB_ic_power:VREG_TL1963A-XX_1.5A_LN_LDO_FAST-TRANSIENT_SOT-223-4_TL1963A-33_1.5A-3.3V
Connections:
- removed net N$24: C12.1, C13.1, C14.1, C15.1, C16.1, C19.1, C20.1, D7.K, LED1.A, SW1.S1, VREG-MCU.VIN, VREG-VIBE.VI
- new net VBAT: C12.1, C13.1, C15.1, C16.1, C19.1, C20.1, D7.K, LED1.A, SW1.S1, VREG-MCU.VIN, VREG-VIBE.VI
- net 3.3V: now also D1.K, D2.K, D3.K, D4.K, D5.K, VIBE1.+, VIBE2.+, VIBE3.+, VIBE4.+, VIBE5.+
- net GND: no longer C14.2
- net VCC: no longer D1.K, D2.K, D3.K, D4.K, D5.K, VIBE1.+, VIBE2.+, VIBE3.+, VIBE4.+, VIBE5.+
